File: mcp73831_bo.sch (EAGLE design)
At the start: 9 parts, among them U1 MCP73831, X1 USBSMD

Commit message: the prog resistor sizing
Parts:
- R1: value 2-7k -> 2-22k (=500-50mA)
Changed lines of the file:
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@@
 <part name="U$4" library="SparkFun-Aesthetics" deviceset="5V" device=""/>
 <part name="C1" library="rcl" deviceset="C-EU" device="C0805" value="4.7uF+"/>
-<part name="R1" library="rcl" deviceset="R-US_" device="M0805" value="2-7k"/>
+<part name="R1" library="rcl" deviceset="R-US_" device="M0805" value="2-22k (=500-50mA)"/>
 </parts>
 <sheets>
